File: ZX-Bus/ZX-Bus.kicad_sch (KiCad schematic)
At the start: 56 parts, among them J1 DIP-40 Pins, J10 DIP14, J11 PBS-4, J12 PBS-5, J2 PLS-3, J3 PLS-6, J4 Power, J5 Main board power, J6 12V, J7 5V, J8 Reset, J9 PLS-2R, U1 Z84C00xxP, U10 27128, U11 74ALS1032, U12 74LS04, U2 74LS245, U3 74LS245, U4 74LS245, U5 74LS245, U6 74ALS1032, U7 74LS253, U8 74LS251, U9 27128

Commit message: ZX-Bus: Describe external connections
/DOS and DOS signal description
Parts:
- added unit 6 of U12
Connections:
- net at J10.12 (Pin_12): now also U12.12; no longer U12.12
- net at J10.13 (Pin_13): now also U12.13; no longer U12.13
Other:
- note added: "~{DOS} - выв. 5 DD7 DOS - выв. 6 DD7"
Changed lines of the file:
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@@
 		(rev "1.0")
+	)
+	(text "~{DOS} - выв. 5 DD7\nDOS - выв. 6 DD7"
+		(exclude_from_sim no)
+		(at 24.13 187.325 0)
+		(effects
+			(font
+				(size 1.27 1.27)
+			)
+		)
 	)
 	(junction
